File: 8051_test.kicad_sch (KiCad schematic)
At the start: 9 parts, among them J1 Conn_01x03_Pin, J2 Conn_01x03_Pin, J3 AVR-ISP-6, U1 8051, X1 TCXO-14, Y1 Crystal

Commit message: Work in progress
Parts:
- added J10, J11, J12, J13, J14, J4, J5, J6, J7, J8, J9: Conn_01x02_Pin, symbol Connector:Conn_01x02_Pin
- added R1, R2, R3, R4, R5, R6, R7, R8: R, symbol Device:R
Connections:
- net +5V: now also R1.2, R2.2, R3.2, R4.2, R5.2, R6.2, R7.2, R8.2
- net AD0: now also J7.2 (Pin_2)
- net AD1: now also J8.2 (Pin_2)
- net AD2: now also J9.2 (Pin_2)
- net AD3: now also J10.2 (Pin_2)
- net AD4: now also J11.2 (Pin_2)
- net AD5: now also J12.2 (Pin_2)
- net AD6: now also J13.2 (Pin_2)
- net AD7: now also J14.2 (Pin_2)
- net MISO: now also J4.2 (Pin_2)
- net MOSI: now also J5.2 (Pin_2)
- net SCK: now also J6.2 (Pin_2)
- new net: J11.1 (Pin_1), R5.1
- new net: J8.1 (Pin_1), R2.1
- new net: J12.1 (Pin_1), R6.1
- new net: J9.1 (Pin_1), R3.1
- new net: J7.1 (Pin_1), R1.1
- new net: J10.1 (Pin_1), R4.1
- new net: J13.1 (Pin_1), R7.1
- new net: J14.1 (Pin_1), R8.1
- new net P1.5: J5.1 (Pin_1)
- new net P1.6: J4.1 (Pin_1)
- new net P1.7: J6.1 (Pin_1)

Commit message: Finished Ver 1.0
Parts:
- removed C3: C, symbol Device:C
- removed J1: Conn_01x03_Pin, Connector_PinHeader_2.54mm:PinHeader_1x03_P2.54mm_Vertical, symbol Connector:Conn_01x03_Pin
- removed J10, J11, J12, J13, J14, J4, J5, J6, J7, J8, J9: Conn_01x02_Pin, symbol Connector:Conn_01x02_Pin
- removed J2: Conn_01x03_Pin, symbol Connector:Conn_01x03_Pin
- removed X1: TCXO-14, Oscillator:Oscillator_DIP-14, symbol Oscillator:TCXO-14
- added C4: 22.0x16V, Capacitor_SMD:C_0603_1608Metric_Pad1.08x0.95mm_HandSolder, symbol Device:C
- added C5: 10.0x16V, Capacitor_SMD:C_0603_1608Metric_Pad1.08x0.95mm_HandSolder, symbol Device:C
- added D1: LED, LED_SMD:LED_0805_2012Metric_Pad1.15x1.40mm_HandSolder, symbol Device:LED
- added DTR1, RST1: Conn_01x02_Pin, Connector_PinHeader_2.54mm:PinHeader_1x02_P2.54mm_Vertical, symbol Connector:Conn_01x02_Pin
- added J17: Prog, Connector_PinHeader_2.54mm:PinHeader_1x06_P2.54mm_Vertical, symbol Connector:Conn_01x06_Socket
- added J2: Pwr, Connector_PinHeader_2.54mm:PinHeader_1x02_P2.54mm_Vertical, symbol Connector:Conn_01x02_Pin
- added J24, J25: Conn_01x20_Pin, Connector_PinHeader_2.54mm:PinHeader_1x20_P2.54mm_Vertical, symbol Connector:Conn_01x20_Pin
- added J4: Conn_02x09_Odd_Even, Connector_PinHeader_2.54mm:PinHeader_2x09_P2.54mm_Vertical, symbol Connector_Generic:Conn_02x09_Odd_Even
- added PwrCon1: Conn_01x03_Pin, Connector_PinHeader_2.54mm:PinHeader_1x03_P2.54mm_Vertical, symbol Connector:Conn_01x03_Pin
- added Q1, Q2: 2N3906, Package_TO_SOT_SMD:SOT-23, symbol Transistor_BJT:2N3906
- added Q3: 2N7000, Package_TO_SOT_SMD:SOT-23, symbol Transistor_FET:2N7000
- added Q4: Conn_02x02_Odd_Even, Connector_PinHeader_2.54mm:PinHeader_2x02_P2.54mm_Vertical, symbol Connector_Generic:Conn_02x02_Odd_Even
- added R10, R11, R16: 2k, Resistor_SMD:R_0603_1608Metric_Pad0.98x0.95mm_HandSolder, symbol Device:R
- added R12, R13: 1k, Resistor_SMD:R_0603_1608Metric_Pad0.98x0.95mm_HandSolder, symbol Device:R
- added R14: 1.1k, Resistor_SMD:R_0603_1608Metric_Pad0.98x0.95mm_HandSolder, symbol Device:R
- added R15: 430, Resistor_SMD:R_0603_1608Metric_Pad0.98x0.95mm_HandSolder, symbol Device:R
- added R17: 5.1k, Resistor_SMD:R_0603_1608Metric_Pad0.98x0.95mm_HandSolder, symbol Device:R
- added R9: 20k, Resistor_SMD:R_0603_1608Metric_Pad0.98x0.95mm_HandSolder, symbol Device:R
- AVR-ISP1: renamed from J3; footprint (none) -> Connector_PinHeader_2.54mm:PinHeader_2x03_P2.54mm_Vertical
- C1, C2: value C -> 22; footprint (none) -> Capacitor_SMD:C_0603_1608Metric_Pad1.08x0.95mm_HandSolder
- R1, R2, R3, R4, R5, R6, R7, R8: value R -> 5.1k; footprint (none) -> Resistor_SMD:R_0603_1608Metric_Pad0.98x0.95mm_HandSolder
- Y1: footprint (none) -> Crystal:Crystal_HC49-U_Vertical
Connections:
- net +5V: now also C4.1, C5.1, J17.4 (Pin_4), J2.2 (Pin_2), PwrCon1.3 (Pin_3), Q1.1 (E), R12.1, R13.1, R17.1
- net A10: now also J25.18 (Pin_18)
- net A11: now also J25.17 (Pin_17)
- net A12: now also J25.16 (Pin_16)
- net A13: now also J25.15 (Pin_15)
- net A14: now also J25.14 (Pin_14)
- net A15: now also J25.13 (Pin_13)
- net A8: now also J25.20 (Pin_20)
- net A9: now also J25.19 (Pin_19)
- net AD0: now also J25.2 (Pin_2), J4.1 (Pin_1)
- net AD1: now also J25.3 (Pin_3), J4.3 (Pin_3)
- net AD2: now also J25.4 (Pin_4), J4.5 (Pin_5)
- net AD3: now also J25.5 (Pin_5), J4.7 (Pin_7)
- net AD4: now also J25.6 (Pin_6), J4.9 (Pin_9)
- net AD5: now also J25.7 (Pin_7), J4.11 (Pin_11)
- net AD6: now also J25.8 (Pin_8), J4.13 (Pin_13)
- net AD7: now also J25.9 (Pin_9), J4.15 (Pin_15)
- net GND: now also C5.2, D1.1 (K), J17.6 (Pin_6), J2.1 (Pin_1), J24.20 (Pin_20), J4.18 (Pin_18), Q2.3 (C), Q3.1 (S), R11.2, R16.2, R9.2
- net MISO: now also J24.7 (Pin_7)
- net MOSI: now also J24.6 (Pin_6)
- net RD: now also J24.17 (Pin_17)
- net RST: now also J24.9 (Pin_9), RST1.1 (Pin_1)
- net SCK: now also J24.8 (Pin_8)
- net VPP: now also J25.1 (Pin_1), PwrCon1.2 (Pin_2)
- net WR: now also J24.16 (Pin_16)
- net X1: now also J24.18 (Pin_18), Q4.2 (Pin_2)
- net X2: now also J24.19 (Pin_19), Q4.4 (Pin_4)
- net at C1.1, Y1.1: now also Q4.1 (Pin_1)
- net at C2.1, Y1.2: now also Q4.3 (Pin_3)
- net at R5.1: now also J4.10 (Pin_10)
- net P1.0: now reaches U1.1 (P1.0/T2)
- net P1.0: now also J24.1 (Pin_1)
- net P3.2: now reaches U1.12 (P3.2/INT0)
- net P3.2: now also J24.12 (Pin_12)
- net P3.3: now reaches U1.13 (P3.3/INT1)
- net P3.3: now also J24.13 (Pin_13)
- net P3.4: now reaches U1.14 (P3.4/T0)
- net P3.4: now also J24.14 (Pin_14)
- net P3.5: now reaches U1.15 (P3.5/T1)
- net P3.5: now also J24.15 (Pin_15)
- net P1.1: now reaches U1.2 (P1.1/T2E)
- net P1.1: now also J24.2 (Pin_2)
- net PSEN: now reaches U1.29 (PSEN)
- net PSEN: now also J25.12 (Pin_12)
- net P1.2: now reaches U1.3 (P1.2)
- net P1.2: now also J24.3 (Pin_3)
- net ALE: now reaches U1.30 (ALE/PROG)
- net ALE: now also J25.11 (Pin_11)
- net EA: now reaches U1.31 (EA/VPP)
- net EA: now also J25.10 (Pin_10), J4.17 (Pin_17), R17.2
- net P1.3: now reaches U1.4 (P1.3)
- net P1.3: now also J24.4 (Pin_4)
- net P1.4: now reaches U1.5 (P1.4)
- net P1.4: now also J24.5 (Pin_5)
- net at R2.1: now also J4.4 (Pin_4)
- net at R6.1: now also J4.12 (Pin_12)
- net at R3.1: now also J4.6 (Pin_6)
- net at R1.1: now also J4.2 (Pin_2)
- net at R4.1: now also J4.8 (Pin_8)
- net at R7.1: now also J4.14 (Pin_14)
- net at R8.1: now also J4.16 (Pin_16)
- net RX renamed P3.0
- net P3.0: now also J17.2 (Pin_2), J24.10 (Pin_10)
- net TX renamed P3.1
- net P3.1: now also J17.3 (Pin_3), J24.11 (Pin_11)
- new net: C4.2, R10.2, R9.1
- new net: DTR1.2 (Pin_2), Q3.2 (G), R15.2, R16.1
- new net: D1.2 (A), R12.2
- new net: Q2.2 (B), R15.1
- new net: R10.1, RST1.2 (Pin_2)
- new net: Q3.3 (D), R14.1
- new net: PwrCon1.1 (Pin_1), Q1.3 (C), Q2.1 (E), R11.1
- new net: Q1.2 (B), R13.2, R14.2
- new net DTR: DTR1.1 (Pin_1), J17.1 (Pin_1)
Other:
- moved on the sheet: C1, C2, R1, R2, R3, R4, R5, R6, R7, R8, Y1

Commit message: Corrected RX/TX pins
Connections:
- net P3.0: now also J17.3 (Pin_3); no longer J17.2 (Pin_2)
- net P3.1: now also J17.2 (Pin_2); no longer J17.3 (Pin_3)

Commit message: Corrected transistors foot print; RX/TX already corrected; ver 1.1
Parts:
- removed Q1, Q2: 2N3906, Package_TO_SOT_SMD:SOT-23, symbol Transistor_BJT:2N3906
- removed Q3: 2N7000, Package_TO_SOT_SMD:SOT-23, symbol Transistor_FET:2N7000
- added Q1, Q2: MMBT3906, Package_TO_SOT_SMD:SOT-23, symbol Transistor_BJT:MMBT3906
- added Q3: 2N7002, Package_TO_SOT_SMD:SOT-23, symbol Transistor_FET:2N7002
Connections:
- net +5V: now also Q1.2 (E)
- net GND: now also Q2.3 (C), Q3.2 (S)
- net at DTR1.2 (Pin_2), R15.2, R16.1: now also Q3.1 (G)
- net at R15.1: now also Q2.1 (B)
- net at R14.1: now also Q3.3 (D)
- net at PwrCon1.1 (Pin_1), R11.1: now also Q1.3 (C), Q2.2 (E)
- net at R13.2, R14.2: now also Q1.1 (B)
Changed lines of the file:
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@@
-	)
-	(symbol
-		(lib_id "Transistor_FET:2N7000")
-		(at 100.33 133.35 0)
-		(unit 1)
-		(exclude_from_sim no)
-		(in_bom yes)
-		(on_board yes)
-		(dnp no)
-		(fields_autoplaced yes)
-		(property "Reference" "Q3"
-			(at 106.68 132.08 0)
-			(effects
-				(font
-					(size 1.27 1.27)
-				)
-				(justify left)
-			)
-		)
-		(property "Value" "2N7000"
-			(at 106.68 134.62 0)
-			(effects
-				(font
-					(size 1.27 1.27)
-				)
-				(justify left)
-			)
-		)
-		(property "Footprint" "Package_TO_SOT_SMD:SOT-23"
-			(at 105.41 135.255 0)
-			(effects
-				(font
-					(size 1.27 1.27)
-					(italic yes)
-				)
-				(justify left)
-				(hide yes)
-			)
-		)
-		(property "Datasheet" "https://www.vishay.com/docs/70226/70226.pdf"
-			(at 100.33 133.35 0)
-			(effects
-				(font
-					(size 1.27 1.27)
-				)
-				(justify left)
-				(hide yes)
-			)
-		)
-		(property "Description" ""
-			(at 100.33 133.35 0)
-			(effects
-				(font
-					(size 1.27 1.27)
-				)
-				(hide yes)
-			)
-		)
-		(pin "1"
-		)
-		(pin "2"
-		)
-		(pin "3"
-		)
-		(instances
-			(project "8051_test"
-				(path "/be4ffa1f-033e-4d23-a6bf-4fadd9d0d171"
-					(reference "Q3")
-					(unit 1)
-				)
-			)
-		)
 	)
 	(symbol
@@
 	)
 	(symbol
-		(lib_id "Transistor_BJT:2N3906")
-		(at 85.725 109.855 90)
-		(unit 1)
-		(exclude_from_sim no)
-		(in_bom yes)
-		(on_board yes)
-		(dnp no)
-		(property "Reference" "Q1"
-			(at 81.915 113.03 90)
-			(effects
-				(font
-					(size 1.27 1.27)
-				)
-			)
-		)
-		(property "Value" "2N3906"
-			(at 91.44 113.03 90)
-			(effects
-				(font
-					(size 1.27 1.27)
-				)
-			)
-		)
-		(property "Footprint" "Package_TO_SOT_SMD:SOT-23"
-			(at 87.63 104.775 0)
-			(effects
-				(font
-					(size 1.27 1.27)
-					(italic yes)
-				)
-				(justify left)
-				(hide yes)
-			)
-		)
-		(property "Datasheet" "https://www.onsemi.com/pub/Collateral/2N3906-D.PDF"
-			(at 85.725 109.855 0)
-			(effects
-				(font
-					(size 1.27 1.27)
-				)
-				(justify left)
-				(hide yes)
-			)
-		)
-		(property "Description" ""
-			(at 85.725 109.855 0)
-			(effects
-				(font
-					(size 1.27 1.27)
-				)
-				(hide yes)
-			)
-		)
-		(pin "1"
-		)
-		(pin "2"
-		)
-		(pin "3"
-		)
-		(instances
-			(project "8051_test"
-				(path "/be4ffa1f-033e-4d23-a6bf-4fadd9d0d171"
-					(reference "Q1")
-					(unit 1)
-				)
-			)
-		)
-	)
-	(symbol
 		(lib_id "Device:R")
 		(at 97.155 119.38 270)
@@
 	)
 	(symbol
+		(lib_id "Transistor_BJT:MMBT3906")
+		(at 85.725 109.855 90)
+		(unit 1)
+		(exclude_from_sim no)
+		(in_bom yes)
+		(on_board yes)
+		(dnp no)
+		(property "Reference" "Q1"
+			(at 81.788 110.236 90)
+			(effects
+				(font
+					(size 1.27 1.27)
+				)
+			)
+		)
+		(property "Value" "MMBT3906"
+			(at 93.98 109.474 90)
+			(effects
+				(font
+					(size 1.27 1.27)
+				)
+			)
+		)
+		(property "Footprint" "Package_TO_SOT_SMD:SOT-23"
+			(at 87.63 104.775 0)
+			(effects
+				(font
+					(size 1.27 1.27)
+					(italic yes)
+				)
+				(justify left)
+				(hide yes)
+			)
+		)
+		(property "Datasheet" "https://www.onsemi.com/pdf/datasheet/pzt3906-d.pdf"
+			(at 85.725 109.855 0)
+			(effects
+				(font
+					(size 1.27 1.27)
+				)
+				(justify left)
+				(hide yes)
+			)
+		)
+		(property "Description" "-0.2A Ic, -40V Vce, Small Signal PNP Transistor, SOT-23"
+			(at 85.725 109.855 0)
+			(effects
+				(font
+					(size 1.27 1.27)
+				)
+				(hide yes)
+			)
+		)
+		(pin "1"
+		)
+		(pin "3"
+		)
+		(pin "2"
+		)
+		(instances
+			(project ""
+				(path "/be4ffa1f-033e-4d23-a6bf-4fadd9d0d171"
+					(reference "Q1")
+					(unit 1)
+				)
+			)
+		)
+	)
+	(symbol
 		(lib_id "Device:R")
 		(at 92.71 34.29 90)
@@
 	)
 	(symbol
+		(lib_id "Transistor_FET:2N7002")
+		(at 100.33 133.35 0)
+		(unit 1)
+		(exclude_from_sim no)
+		(in_bom yes)
+		(on_board yes)
+		(dnp no)
+		(fields_autoplaced yes)
+		(property "Reference" "Q3"
+			(at 106.68 132.0799 0)
+			(effects
+				(font
+					(size 1.27 1.27)
+				)
+				(justify left)
+			)
+		)
+		(property "Value" "2N7002"
+			(at 106.68 134.6199 0)
+			(effects
+				(font
+					(size 1.27 1.27)
+				)
+				(justify left)
+			)
+		)
+		(property "Footprint" "Package_TO_SOT_SMD:SOT-23"
+			(at 105.41 135.255 0)
+			(effects
+				(font
+					(size 1.27 1.27)
+					(italic yes)
+				)
+				(justify left)
+				(hide yes)
+			)
+		)
+		(property "Datasheet" "https://www.onsemi.com/pub/Collateral/NDS7002A-D.PDF"
+			(at 105.41 137.16 0)
+			(effects
+				(font
+					(size 1.27 1.27)
+				)
+				(justify left)
+				(hide yes)
+			)
+		)
+		(property "Description" "0.115A Id, 60V Vds, N-Channel MOSFET, SOT-23"
+			(at 100.33 133.35 0)
+			(effects
+				(font
+					(size 1.27 1.27)
+				)
+				(hide yes)
+			)
+		)
+		(pin "1"
+		)
+		(pin "3"
+		)
+		(pin "2"
+		)
+		(instances
+			(project ""
+				(path "/be4ffa1f-033e-4d23-a6bf-4fadd9d0d171"
+					(reference "Q3")
+					(unit 1)
+				)
+			)
+		)
+	)
+	(symbol
 		(lib_id "Device:R")
 		(at 70.485 43.18 180)
@@
 	)
 	(symbol
-		(lib_id "Transistor_BJT:2N3906")
+		(lib_id "Transistor_BJT:MMBT3906")
 		(at 81.28 125.095 180)
 		(unit 1)
@@
 		(on_board yes)
 		(dnp no)
-		(fields_autoplaced yes)
 		(property "Reference" "Q2"
-			(at 75.565 123.825 0)
+			(at 75.565 123.8249 0)
 			(effects
 				(font
@@
 			)
 		)
-		(property "Value" "2N3906"
-			(at 75.565 126.365 0)
+		(property "Value" "MMBT3906"
+			(at 75.946 126.746 0)
 			(effects
 				(font
@@
 			)
 		)
-		(property "Datasheet" "https://www.onsemi.com/pub/Collateral/2N3906-D.PDF"
+		(property "Datasheet" "https://www.onsemi.com/pdf/datasheet/pzt3906-d.pdf"
 			(at 81.28 125.095 0)
 			(effects
@@
 			)
 		)
-		(property "Description" ""
+		(property "Description" "-0.2A Ic, -40V Vce, Small Signal PNP Transistor, SOT-23"
 			(at 81.28 125.095 0)
 			(effects
@@
 		(pin "1"
 		)
+		(pin "3"
+		)
 		(pin "2"
 		)
-		(pin "3"
-		)
-		(instances
-			(project "8051_test"
+		(instances
+			(project ""
 				(path "/be4ffa1f-033e-4d23-a6bf-4fadd9d0d171"
 					(reference "Q2")

Commit message: Updated to next version using ZIF socket
Parts:
- removed PwrCon1: Conn_01x03_Pin, Connector_PinHeader_2.54mm:PinHeader_1x03_P2.54mm_Vertical, symbol Connector:Conn_01x03_Pin
- added J1: GND, Connector_PinHeader_2.54mm:PinHeader_1x02_P2.54mm_Vertical, symbol Connector:Conn_01x02_Pin
- added J3: PL2, Connector_PinHeader_2.54mm:PinHeader_1x20_P2.54mm_Vertical, symbol Connector:Conn_01x20_Pin
- added J5: PR2, Connector_PinHeader_2.54mm:PinHeader_1x20_P2.54mm_Vertical, symbol Connector:Conn_01x20_Pin
- added SW1: SW_SPDT, Button_Switch_THT:SPDT_Omron_D2F_5pins, symbol Switch:SW_SPDT
- AVR-ISP1: footprint Connector_PinHeader_2.54mm:PinHeader_2x03_P2.54mm_Vertical -> Connector_IDC:IDC-Header_2x03_P2.54mm_Vertical
- DTR1: value Conn_01x02_Pin -> Prog
- J17: value Prog -> UART
- J2: value Pwr -> +5V
- J24: value Conn_01x20_Pin -> PL1
- J25: value Conn_01x20_Pin -> PR1
- J4: value Conn_02x09_Odd_Even -> Rs
- Q4: value Conn_02x02_Odd_Even -> Conn Crystal
- RST1: value Conn_01x02_Pin -> Reset
- U1: footprint Package_DIP:DIP-40_W15.24mm_Socket_LongPads -> Socket:DIP_Socket-40_W11.9_W12.7_W15.24_W17.78_W18.5_3M_240-1280-00-0602J
- Y1: value Crystal -> 11.0592
Connections:
- net +5V: now also J2.1 (Pin_1), SW1.1 (A)
- net A10: now also J5.18 (Pin_18)
- net A11: now also J5.17 (Pin_17)
- net A12: now also J5.16 (Pin_16)
- net A13: now also J5.15 (Pin_15)
- net A14: now also J5.14 (Pin_14)
- net A15: now also J5.13 (Pin_13)
- net A8: now also J5.20 (Pin_20)
- net A9: now also J5.19 (Pin_19)
- net AD0: now also J5.2 (Pin_2)
- net AD1: now also J5.3 (Pin_3)
- net AD2: now also J5.4 (Pin_4)
- net AD3: now also J5.5 (Pin_5)
- net AD4: now also J5.6 (Pin_6)
- net AD5: now also J5.7 (Pin_7)
- net AD6: now also J5.8 (Pin_8)
- net AD7: now also J5.9 (Pin_9)
- net ALE: now also J5.11 (Pin_11)
- net EA: now also J5.10 (Pin_10)
- net GND: now also J1.1 (Pin_1), J1.2 (Pin_2), J3.20 (Pin_20); no longer J2.1 (Pin_1)
- net MISO: now also J3.7 (Pin_7)
- net MOSI: now also J3.6 (Pin_6)
- net P1.0: now also J3.1 (Pin_1)
- net P1.1: now also J3.2 (Pin_2)
- net P1.2: now also J3.3 (Pin_3)
- net P1.3: now also J3.4 (Pin_4)
- net P1.4: now also J3.5 (Pin_5)
- net P3.0: now also J3.10 (Pin_10)
- net P3.1: now also J3.11 (Pin_11)
- net P3.2: now also J3.12 (Pin_12)
- net P3.3: now also J3.13 (Pin_13)
- net P3.4: now also J3.14 (Pin_14)
- net P3.5: now also J3.15 (Pin_15)
- net PSEN: now also J5.12 (Pin_12)
- net RST: now also J3.9 (Pin_9)
- net SCK: now also J3.8 (Pin_8)
- net VPP: now also J5.1 (Pin_1), SW1.2 (B)
- net X1: now also J3.18 (Pin_18)
- net X2: now also J3.19 (Pin_19)
- net at Q1.3 (C), Q2.2 (E), R11.1: now also SW1.3 (C)
- net RD renamed ~{RD}
- net ~{RD}: now also J3.17 (Pin_17)
- net WR renamed ~{WR}
- net ~{WR}: now also J3.16 (Pin_16)
Other:
- moved on the sheet: C4, J2, J24, J25, R10, R9, RST1
