File: 8051header.kicad_pcb (KiCad board)
At the start: 2 copper layers, 56 x 70 mm, 40 parts, among them J1 GND, J17 UART, J2 +5V, J24 PL1, J25 PR1, J3 PL2, J4 Rs, J5 PR2, Q1 MMBT3906, Q2 MMBT3906, Q3 2N7002, Q4 Conn Crystal, SW1 SW_SPDT, U1 8051, Y1 11.0592

Commit message: Added github reference
Other:
- board text added: "https://github.com/afiglee/8051header"
Changed lines of the file:
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@@
 		(layer "Edge.Cuts")
+	)
+	(gr_text "https://github.com/afiglee/8051header"
+		(at 111.125 114.173 0)
+		(layer "B.Cu")
+		(effects
+			(font
+				(size 1.5 1.5)
+				(thickness 0.3)
+				(bold yes)
+			)
+			(justify left bottom mirror)
+		)
 	)
 	(gr_text "AT89S52/STC89C52"
